File: MRF49XA.brd (EAGLE design)
At the start: 43 x 31.4 mm, 47 parts, among them J1 AVR_SPI_PRG_6NS, Q1 10Mhz, U1 ATSHA204, U2 ANT1204F002R0433A, U3 V_REG_LDOSMD, U4 MCP73831, Y1 16MHZ

Commit message: BOM
Added BOM and values to antenna section
Parts:
- C5: value (none) -> 1.2pF
- C6: value (none) -> 27pF
- C9: value (none) -> 2.7pF
- L1: value (none) -> 100nH
- L2: value (none) -> 8.2nH
- L3: value (none) -> 22nH
Changed lines of the file:
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@@
 <attribute name="VALUE" x="17.9475" y="23.0125" size="0.6096" layer="27"/>
 </element>
-<element name="L2" library="SparkFun-Passives" package="0603" value="" x="35.8" y="15.3" smashed="yes" rot="R270">
+<element name="L2" library="SparkFun-Passives" package="0603" value="8.2nH" x="35.8" y="15.3" smashed="yes" rot="R270">
 <attribute name="NAME" x="36.662" y="13.789" size="0.6096" layer="25" font="vector" rot="R270"/>
 <attribute name="VALUE" x="34.657" y="16.316" size="0.4064" layer="27" font="vector" rot="R270"/>
 </element>
-<element name="L1" library="SparkFun-Passives" package="0603" value="" x="35.8" y="18.7" smashed="yes" rot="R270">
+<element name="L1" library="SparkFun-Passives" package="0603" value="100nH" x="35.8" y="18.7" smashed="yes" rot="R270">
 <attribute name="NAME" x="35.462" y="21.489" size="0.6096" layer="25" font="vector" rot="R270"/>
 <attribute name="VALUE" x="34.657" y="19.716" size="0.4064" layer="27" font="vector" rot="R270"/>
 </element>
-<element name="L3" library="SparkFun-Passives" package="0603" value="" x="38.1" y="16.2" smashed="yes" rot="R180">
+<element name="L3" library="SparkFun-Passives" package="0603" value="22nH" x="38.1" y="16.2" smashed="yes" rot="R180">
 <attribute name="NAME" x="37.589" y="15.438" size="0.6096" layer="25" font="vector" rot="R180"/>
 <attribute name="VALUE" x="39.116" y="17.343" size="0.4064" layer="27" font="vector" rot="R180"/>
 </element>
-<element name="C5" library="SparkFun-Passives" package="0603-CAP" value="" x="38.1" y="17.8" smashed="yes">
+<element name="C5" library="SparkFun-Passives" package="0603-CAP" value="1.2pF" x="38.1" y="17.8" smashed="yes">
 <attribute name="NAME" x="37.611" y="18.562" size="0.6096" layer="25" font="vector"/>
 <attribute name="VALUE" x="37.084" y="16.657" size="0.4064" layer="27" font="vector"/>
 </element>
-<element name="C6" library="SparkFun-Passives" package="0603-CAP" value="" x="40.5" y="17" smashed="yes" rot="R270">
+<element name="C6" library="SparkFun-Passives" package="0603-CAP" value="27pF" x="40.5" y="17" smashed="yes" rot="R270">
 <attribute name="NAME" x="41.262" y="16.889" size="0.6096" layer="25" font="vector"/>
 <attribute name="VALUE" x="39.357" y="18.016" size="0.4064" layer="27" font="vector" rot="R270"/>
 </element>
-<element name="C9" library="SparkFun-Passives" package="0603-CAP" value="" x="35.8" y="11.9" smashed="yes" rot="R270">
+<element name="C9" library="SparkFun-Passives" package="0603-CAP" value="2.7pF" x="35.8" y="11.9" smashed="yes" rot="R270">
 <attribute name="NAME" x="35.662" y="10.289" size="0.6096" layer="25" font="vector" rot="R270"/>
 <attribute name="VALUE" x="34.657" y="12.916" size="0.4064" layer="27" font="vector" rot="R270"/>
